File: smart_pouch.kicad_sch (KiCad schematic)
At the start: 12 parts, among them CN1 B2B-PH-K-S, U1 nRF52840, U2 NRF9151-LACA-R7, U3 NPM1300-CAAA-R7, U4 BMA400, U5 BWU.FL-IPEX1, U6 BWU.FL-IPEX1, U7 MT3608, U8 SM06B-SRSS-TB

Commit message: hella
Parts:
- removed Card1: SMN-303, easyeda2kicad:SIM-SMD_SMN-303, symbol easyeda2kicad:SMN-303
- removed D1: PRTR5V0U2X_C2827688, easyeda2kicad:SOT-143-4_L2.9-W1.3-P1.92-LS2.4-BL, symbol easyeda2kicad:PRTR5V0U2X_C2827688
- removed U5: BWU.FL-IPEX1, easyeda2kicad:IPEX-SMD_BWIPX-1-001E, symbol easyeda2kicad:BWU.FL-IPEX1
- removed U7: MT3608, easyeda2kicad:SOT-23-6_L2.9-W1.6-P0.95-LS2.8-BL, symbol easyeda2kicad:MT3608
- removed USB1: TYPE-C 6P, Connector_USB:USB_C_Receptacle_GCT_USB4125-xx-x-0190_6P_TopMnt_Horizontal, symbol easyeda2kicad:TYPE-C6P
- added C1, C12, C13, C14, C15, C29, C30, C31, C4, C6, C8: 100nF, symbol Device:C
- added C10, C16, C18: 10u, symbol Device:C
- added C11, C2, C24, C3, C5: 1uF, symbol Device:C
- added C17, C19, C9: 22u 25V, symbol Device:C
- added C20, C21, C22, C23, C7: 10uF, symbol Device:C
- added C25: 0.5uF, symbol Device:C
- added C26: 0.8uF, symbol Device:C
- added C27, C28: 12pF, symbol Device:C
- added D1, D10, D11, D12, D6, D7, D8, D9: LED, symbol Device:LED
- added D13, D14, D15, D4: SS34_C8678, easyeda2kicad:SMA_L4.3-W2.6-LS5.2-RD, symbol easyeda2kicad:SS34_C8678
- added D3: SP3012-04UTG, easyeda2kicad:UDFN-10_L2.5-W1.0-P0.50-BL, symbol easyeda2kicad:SP3012-04UTG
- added D5: PRTR5V0U2X, Package_TO_SOT_SMD:SOT-143, symbol Power_Protection:PRTR5V0U2X
- added J1: Conn_01x02_Pin, symbol Connector:Conn_01x02_Pin
- added J2: Conn_01x03_Pin, symbol Connector:Conn_01x03_Pin
- added J3: SIM_Card, symbol Connector:SIM_Card
- added L1, L2, L3: 10uH, symbol Device:L
- added L4, L5: 2.2uH, symbol Device:L
- added L6: 4.7nH, symbol Device:L
- added LED1: 19-237/R6GHBHC-A01/2T, easyeda2kicad:LED-ARRAY-SMD_4P-L1.6-W1.6-BL_1, symbol easyeda2kicad:19-237_R6GHBHC-A01_2T
- added P1: USB_C_Plug_USB2.0, symbol Connector:USB_C_Plug_USB2.0
- added Q1, Q2, Q4: BSS84, Package_TO_SOT_SMD:SOT-23, symbol Transistor_FET:BSS84
- added Q3, Q5, Q6: 2N7002, Package_TO_SOT_SMD:SOT-23, symbol Transistor_FET:2N7002
- added R1: 47k, symbol Device:R
- added R10, R11, R12, R13, R14, R7, R8, R9: 4.7, symbol Device:R
- added R15: 5.1k, symbol Device:R
- added R16, R17: 22R, symbol Device:R
- added R18, R23, R24: 100R, symbol Device:R
- added R19: 191k, symbol Device:R
- added R2: 150k, symbol Device:R
- added R20, R22, R3, R4, R6: 10k, symbol Device:R
- added R21: 240k, symbol Device:R
- added R5: 73.2k, symbol Device:R
- added RV1: R_Potentiometer_Trim, symbol Device:R_Potentiometer_Trim
- added SW2: SW_SPST, symbol Switch:SW_SPST
- added TH1: Thermistor, symbol Device:Thermistor
- added U10: BWU.FL-IPEX1, easyeda2kicad:IPEX-SMD_BWIPX-1-001E, symbol easyeda2kicad:BWU.FL-IPEX1
- added U11, U14: ZX-PZ1.27-2-5PZZ, easyeda2kicad:HDR-TH_10P-P1.27-V-M-R2-C5-S1.27, symbol easyeda2kicad:ZX-PZ1.27-2-5PZZ
- added U12, U13, U5: MT3608, easyeda2kicad:SOT-23-6_L2.9-W1.6-P0.95-LS2.8-BL, symbol easyeda2kicad:MT3608
- added U7: AN6520-245, easyeda2kicad:ANT-SMD_L6.5-W2.0, symbol easyeda2kicad:AN6520-245
- added U9: B4B-XH-A, easyeda2kicad:CONN-TH_B4B-XH-A-LF-SN, symbol easyeda2kicad:B4B-XH-A
- added Y1: 32MHz, symbol Device:Crystal
Connections:
- net GND: now also CN1.2, U1.B7 (VSS), U1.EP (VSS), U1.F23 (VSS_PA), U2.25 (GND), U2.36 (GND), U3.A6 (AVSS), U3.A7 (PVSS1), U3.E7 (PVSS2), U4.1 (SDO), U4.8 (GNDIO), U6.2, U6.3, U8.1, C10.2, C11.1, C12.1, C13.1, C14.1, C15.1, C16.2, C17.2, C18.2, C19.2, C2.1, C20.2, C21.2, C22.2, C23.1, C24.1, C25.1, C26.1, C27.2, C28.2, C29.1, C3.2, C30.1, C31.1, C4.2, C5.2, C6.2, C7.1, C8.1, C9.2, D3.3 (GND), D3.8 (GND), D5.1 (GND), J3.5 (GND), P1.A1 (GND), P1.A12 (GND), P1.B1 (GND), P1.B12 (GND), P1.SH (SHIELD), Q3.2 (S), Q5.2 (S), Q6.2 (S), R1.2, R10.2, R11.2, R12.2, R13.2, R14.2, R15.2, R2.2, R20.2, R22.2, R6.2, R7.2, R8.2, R9.2, RV1.3, SW2.2 (B), TH1.2, U10.2, U10.3, U11.3, U11.5, U11.9, U12.2 (GND), U13.2 (GND), U14.3, U14.5, U14.9, U5.2 (GND), U7.2, U9.1
- net CELL: now reaches U6.1
- net CELL: now also U2.35 (ANT)
- net SIREN_PWM: now reaches U2.10 (ENABLE)
- net SIREN_PWM: now also U1.AD20 (P0.24), U2.14 (VDD), U3.C1 (VSYS), U3.C2 (VSYS), U3.C7 (PVDD), C20.1, C21.1, C22.1, LED1.4 (+), R23.1
- net SIM_RST: now reaches U2.16 (SIM_RST)
- net SIM_RST: now also D3.7
- net SIM_IO: now reaches U2.17 (SIM_IO)
- net SIM_IO: now also D3.10
- net SIM_CLK: now reaches U2.18 (SIM_CLK)
- net SIM_CLK: now also D3.9
- net SIM_1V8: now reaches U2.19 (SIM_1V8)
- net SIM_1V8: now also D3.6
- net at U2.24 (DEC0): now also C31.2
- net SWDCLK_9151: now reaches U2.3 (SWDCLK)
- net SWDIO_9151: now reaches U2.4 (SWDIO)
- net GNSS: now reaches U2.42 (GPS)
- net GNSS: now also U10.1
- net VCC_9151: now reaches U2.65 (VDD_GPIO)
- net VCC_9151: now also C29.2, C30.2, U11.1
- net UART_RX: now reaches U2.77 (P0.16)
- net UART_RX: now also U1.AD8 (P0.13)
- net UART_TX: now reaches U2.78 (P0.17)
- net UART_TX: now also U1.U1 (TRACEDATA1/P0.12)
- net SWO_9151: now reaches U2.79 (P0.18)
- net nRST_9151: now reaches U2.9 (nRESET)
- net nRST_9151: now also U11.10
- net +1V8: now reaches U4.10 (CSB)
- net +1V8: now also U1.A22 (VDD), U1.AD14 (VDD), U1.AD23 (VDD), U1.B1 (VDD), U1.W1 (VDD), U1.Y2 (VDDH), U3.B6 (VOUT1), U3.E4 (VDDIO), U4.3 (VDDIO), U4.7 (VDD), U8.4, C2.2, C6.1, C7.2, L4.1, R3.2, R4.2
- net ACC_SCL: now reaches U4.12 (SCX)
- net ACC_SCL: now also U1.AC15 (P0.19)
- net ACC_SDA: now reaches U4.2 (SDX)
- net ACC_SDA: now also U1.AD12 (P0.17)
- net ACC_INT1: now reaches U4.5 (INT1)
- net ACC_INT1: now also U1.AD16 (P0.20)
- net ACC_INT2: now reaches U4.6 (INT2)
- net ACC_INT2: now also U1.AC17 (P0.21)
- net at U3.A1 (LED0): now also LED1.1 (R-)
- net at U3.A2 (LED1): now also LED1.2 (G-)
- net at U3.A3 (LED2): now also LED1.3 (B-)
- net BIO_LS: now reaches U3.A4 (LSOUT1/VOUTLDO1)
- net BIO_LS: now also U8.6
- net SEN_IRQ: now reaches U3.B1 (VBUS)
- net SEN_IRQ: now also U1.AD2 (VBUS), U3.B2 (VBUS), U8.5, C24.2, C3.1, C4.1, C5.1, D5.4 (VCC), P1.A4 (VBUS), P1.A9 (VBUS), P1.B4 (VBUS), P1.B9 (VBUS)
- net +3.3V: now reaches U3.B4 (LSIN1/VINLDO1)
- net +3.3V: now also U3.D7 (SW2), C23.2, L5.1
- net at U3.B7 (SW1): now also L4.2
- net at U3.C6 (VOUT2): now also L5.2
- net at U3.D1 (VBAT): now also U3.D2 (VBAT)
- net at U3.D3 (NTC): now also TH1.1
- net RESET: now reaches U3.D6 (GPIO0)
- net RESET: now also SW2.1 (A)
- net at U3.E1 (VSET2): now also R2.1
- net at U3.E2 (VSET1): now also R1.1
- net NPM_SCL: now reaches U3.E3 (SCL)
- net NPM_SCL: now also U1.AD10 (P0.15)
- net NPM_SDA: now reaches U3.E5 (SDA)
- net NPM_SDA: now also U1.AC9 (P0.14)
- net NPM_INT: now reaches U3.E6 (GPIO1)
- net NPM_INT: now also U1.AC11 (P0.16)
- net at U1.A23 (XC2): now also C28.1, Y1.1
- net SWDCLK_52840: now reaches U1.AA24 (SWDCLK)
- net SWDCLK_52840: now also U14.4
- net nRST_52840: now reaches U1.AC13 (P0.18/~{RESET})
- net nRST_52840: now also U14.10
- net SIREN_FB: now reaches U1.AC19 (P0.23)
- net SIREN_FB: now also RV1.1
- net SIREN_PWM_INVERTED: now reaches U1.AC21 (P0.25)
- net SIREN_PWM_INVERTED: now also R24.2
- net SWDIO_52840: now reaches U1.AC24 (SWDIO)
- net SWDIO_52840: now also U14.2
- net at U1.AC5 (DECUSB): now also C15.2
- net Strobe_In: now reaches U1.AD18 (P0.22)
- net Strobe_In: now also Q1.1 (G)
- net SWO_52840: now reaches U1.AD22 (TRACEDATA0/P1.00)
- net SWO_52840: now also U14.6
- net USB_D-: now reaches U1.AD4 (D-)
- net USB_D-: now also D5.3 (I/O2), R17.2
- net USB_D+: now reaches U1.AD6 (D+)
- net USB_D+: now also D5.2 (I/O1), R16.2
- net at U1.B24 (XC1): now also C27.1, Y1.2
- net at U1.B5 (DEC4): now also C12.2
- net at U1.C1 (DEC1): now also C8.2
- net at U1.D23 (DEC3): now also C11.2
- net at U1.E24 (DEC6): now also C14.2
- net SEN_TX: now reaches U1.G1 (P0.26)
- net SEN_TX: now also U8.3
- net SEN_RX: now reaches U1.H2 (P0.27)
- net SEN_RX: now also U8.2
- net at U1.H23 (ANT): now also C25.2, L6.2
- net at U1.N24 (DEC5): now also C13.2
- new net: C1.1, D3.1
- new net: C1.2, J3.1 (VCC)
- new net: D13.2 (A), J1.2 (Pin_2), Q3.3 (D)
- new net: R19.2, R20.1, U12.3 (FB)
- new net: Q2.1 (G), Q5.1 (G), R23.2
- new net: J2.1 (Pin_1), Q2.3 (D), Q5.3 (D)
- new net: D9.1 (K), R11.1
- new net: C10.1, L1.1, U5.4 (EN), U5.5 (IN)
- new net: D4.2 (A), L1.2, U5.1 (SW)
- new net: D8.1 (K), R10.1
- new net: C26.2, L6.1, U7.1
- new net: D10.1 (K), R12.1
- new net: P1.A5 (CC), R15.1
- new net: P1.A6 (D+), R16.1
- new net: P1.A7 (D-), R17.1
- new net: D3.5, J3.7 (I/O), R4.1
- new net: Q4.1 (G), Q6.1 (G), R24.1
- new net: J2.3 (Pin_3), Q4.3 (D), Q6.3 (D)
- new net: C16.1, L2.1, U12.4 (EN), U12.5 (IN)
- new net: J2.2 (Pin_2), RV1.2
- new net: D14.2 (A), L2.2, U12.1 (SW)
- new net: D1.2 (A), D10.2 (A), D11.2 (A), D12.2 (A), D6.2 (A), D7.2 (A), D8.2 (A), D9.2 (A), Q1.2 (S)
- new net: D3.2, J3.2 (RST)
- new net: D3.4, J3.3 (CLK), R3.1
- new net: R21.2, R22.1, U13.3 (FB)
- new net: C18.1, L3.1, U13.4 (EN), U13.5 (IN)
- new net: R5.2, R6.1, U5.3 (FB)
- new net: D1.1 (K), R7.1
- new net: D7.1 (K), R9.1
- new net: D6.1 (K), R8.1
- new net: Q3.1 (G), R18.2
- new net: D12.1 (K), R14.1
- new net: D11.1 (K), R13.1
- new net: D15.2 (A), L3.2, U13.1 (SW)
- new net +12V: C17.1, D13.1 (K), D14.1 (K), J1.1 (Pin_1), R19.1
- new net +15V: C19.1, D15.1 (K), Q2.2 (S), Q4.2 (S), R21.1
- new net +5V: C9.1, D4.1 (K), Q1.3 (D), R5.1
- new net RX_9151: U9.4
- new net Solenoid: R18.1
- new net TX_9151: U9.3
- new net VCC: U9.2
- new net VCC_52840: U14.1
- no-connect marks 27 -> 122
Other:
- note added: "+"
- note added: "-"
- note added: "3.7V"
- note added: "3608 Boost Circuit 12V"
- note added: "3608 Boost Circuit 30V"
- note added: "3608 Boost Circuit 5V"
- note added: "52840 SWD"
- note added: "9151 SWD"
- note added: "9151 UART"
- note added: "ACC"
- note added: "Accelerometer"
- note added: "Battery JST 2.54mm 1x2P"
- note added: "Biometric"
- note added: "Biometric UART"
- note added: "External Connections"
- note added: "FB"
- note added: "NRF9151 LTE-M + GNSS"
- note added: "PMIC"
- note added: "Piezo"
- note added: "Power"
- note added: "SIM"
- note added: "SWD 52840"
- note added: "SWD 9151"
- note added: "Sensors"
- note added: "Sim Card"
- note added: "Siren"
- note added: "Solenoid"
- note added: "Status LED"
- note added: "Strobe"
- note added: "Strobe Light"
- note added: "USB-C"
- note added: "nRF52840 BLE"
- note added: "npm1300"
- note added: "u.FL Antenna"
- moved on the sheet: CN1, U1, U2, U3, U4, U6, U8
