File: smart_pouch.kicad_sch (KiCad schematic)
At the start: 105 parts, among them CN1 B2B-PH-K-S, J1 Conn_01x02_Pin, J2 Conn_01x03_Pin, J3 SIM_Card, P1 USB_C_Plug_USB2.0, Q1 BSS84, Q2 BSS84, Q3 2N7002, Q4 BSS84, Q5 2N7002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

Commit message: final claude update
Parts:
- added LED2: 19-237/R6GHBHC-A01/2T, easyeda2kicad:LED-ARRAY-SMD_4P-L1.6-W1.6-BL_1, symbol easyeda2kicad:19-237_R6GHBHC-A01_2T
- added R28, R5, R6: 330, symbol Device:R
Connections:
- net VSYS: now also LED2.4 (+)
- net at U1.A10 (AIN5/P0.29): now also R6.1
- net at U1.B11 (AIN4/P0.28): now also R5.1
- net at U1.B9 (AIN6/P0.30): now also R28.1
- new net: LED2.1 (R-), R28.2
- new net: LED2.2 (G-), R6.2
- new net: LED2.3 (B-), R5.2
- no-connect marks 117 -> 113
Other:
- note removed: "3608 Boost Circuit 5V"
- moved on the sheet: C1, C11, C12, C13, C14, C15, C16, C17, C18, C19, C2, C20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

Commit message: codex run
Parts:
- removed C28, C34: 12pF, Capacitor_SMD:C_0402_1005Metric, symbol Device:C
- removed SW2: SW_SPST, Button_Switch_SMD:SW_SPST_PTS645, symbol Switch:SW_SPST
- added SW1: SW_Push, symbol Switch:SW_Push
- U2: footprint easyeda2kicad:LGA-113_L12.1-W11.1_NRF9151-SICA -> easyeda2kicad:LGA-113_L12.1-W11.1_NRF9151-LACA-R7
- U3: value NPM1300-CAAA-R7 -> NPM1300
- U8: value SM06B-SRSS-TB -> SEN0348_CONN
Connections:
- net RESET is gone; now on net NPM_RESET: U3.D6 (GPIO0)
- net RX_9151 is gone; now on net UART_RX: U9.4
- net TX_9151 is gone; now on net UART_TX: U9.3
- net VCC is gone; now on net +1V8: U9.2
- net VCC_52840 is gone; now on net +3.3V: U14.1
- net VCC_9151 is gone; now on net +1V8: U11.1
- net +1V8: now also C32.2, U2.29 (VIO)
- net GND: now also SW1.2
- net SEN_IRQ: now also U1.V23 (P1.03)
- net SIM_1V8: now also C1.2, J3.1 (VCC)
- net SIM_CLK: now also D3.4, J3.3 (CLK), R3.1
- net SIM_IO: now also D3.5, J3.7 (I/O), R4.1
- net SIM_RST: now also D3.2, J3.2 (RST)
- net Solenoid: now also U1.W24 (P1.02)
- net VSYS: no longer U3.D4 (SHPHLD)
- net at U3.D1 (VBAT): no longer U3.D2 (VBAT)
- net NPM_RESET: now reaches U1.Y23 (P1.01)
- net USB_5V renamed +5V
- new net: SW1.1, U3.D4 (SHPHLD)
- no-connect marks 113 -> 110

Commit message: BOM update
Parts:
- C25: value 0.5uF -> 0.6pF
- C26: value 0.8uF -> 0.8pF
- CN1: value B2B-PH-K-S -> B2B-PH-SM4-TB; footprint easyeda2kicad:CONN-TH_B2B-PH-K-S -> easyeda2kicad:CONN-SMD_B2B-PH-SM4-TB-LF-SN; LCSC Part C131337 -> C160352; MPN B2B-PH-K-S(LF)(SN) -> B2B-PH-SM4-TB(LF)(SN)
- J1: value Conn_01x02_Pin -> XH-2P-SMD; footprint Connector_PinHeader_2.54mm:PinHeader_1x02_P2.54mm_Vertical -> easyeda2kicad:CONN-SMD_2P-P2.54_XH2.54-2AB
- J2: value Conn_01x03_Pin -> 2.54-3P-LT; footprint Connector_PinHeader_2.54mm:PinHeader_1x03_P2.54mm_Vertical -> easyeda2kicad:CONN-SMD_2.54-3P-LT
- L2, L3: footprint easyeda2kicad:IND-SMD_L4.0-W4.0_LQH44PN2R2MP0L -> easyeda2kicad:IND-SMD_L4.0-W4.0
- L4, L5: footprint easyeda2kicad:IND-SMD_L4.0-W4.0_LQH44PN2R2MP0L -> easyeda2kicad:IND-SMD_L4.0-W4.0_NRS4018T
- L6: footprint easyeda2kicad:IND-SMD_L4.0-W4.0_LQH44PN2R2MP0L -> easyeda2kicad:L0402-R-RD
- R28, R5, R6: footprint (none) -> Resistor_SMD:R_0402_1005Metric
- RV1: value R_Potentiometer_Trim -> 10k; footprint Potentiometer_THT:Potentiometer_Bourns_3296W_Vertical -> easyeda2kicad:RES-ADJ-SMD_3P-L3.0-W3.8-P1.75-BR
- SW1: footprint (none) -> easyeda2kicad:KEY-SMD_4P-L4.2-W3.2-P2.20-LS4.6
- U11, U14: value ZX-PZ1.27-2-5PZZ -> HX PZ1.27-2x5P TP; footprint easyeda2kicad:HDR-TH_10P-P1.27-V-M-R2-C5-S1.27 -> easyeda2kicad:HDR-SMD_10P-P1.27-V-M-R2-C5-LS5.5_1; LCSC Part C7501289 -> C41376037; MPN ZX-PZ1.27-2-5PZZ -> HX PZ1.27-2x5P TP; Manufacturer Megastar(兆星) -> hanxia
- U2: value NRF9151-SICA -> NRF9151-LACA-R7
- U9: value B4B-XH-A -> SM04B-SRSS-TB; footprint easyeda2kicad:CONN-TH_B4B-XH-A-LF-SN -> easyeda2kicad:CONN-SMD_4P-P1.00_SM04B-SRSS-TB-LF-SN; LCSC Part C144395 -> C160404; MPN B4B-XH-A(LF)(SN) -> SM04B-SRSS-TB(LF)(SN)
Changed lines of the file:
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@@
 			)
 		)
-		(property "Footprint" ""
+		(property "Footprint" "easyeda2kicad:KEY-SMD_4P-L4.2-W3.2-P2.20-LS4.6"
 			(at 518.16 185.42 0)
 			(hide yes)
@@
 			)
 		)
-		(property "Value" "Conn_01x02_Pin"
+		(property "Value" "XH-2P-SMD"
 			(at 271.78 66.04 0)
 			(show_name no)
@@
 			)
 		)
-		(property "Footprint" "Connector_PinHeader_2.54mm:PinHeader_1x02_P2.54mm_Vertical"
+		(property "Footprint" "easyeda2kicad:CONN-SMD_2P-P2.54_XH2.54-2AB"
 			(at 267.97 69.85 0)
 			(hide yes)
@@
 			)
 		)
-		(property "Value" "NRF9151-SICA"
+		(property "Value" "NRF9151-LACA-R7"
 			(at 95.25 156.21 0)
 			(show_name no)
@@
 			)
 		)
-		(property "Value" "B2B-PH-K-S"
+		(property "Value" "B2B-PH-SM4-TB"
 			(at 168.91 78.74 0)
 			(show_name no)
@@
 			)
 		)
-		(property "Footprint" "easyeda2kicad:CONN-TH_B2B-PH-K-S"
+		(property "Footprint" "easyeda2kicad:CONN-SMD_B2B-PH-SM4-TB-LF-SN"
 			(at 171.45 96.52 0)
 			(hide yes)
@@
 			)
 		)
-		(property "Datasheet" "https://lcsc.com/product-detail/PH-Connectors_JST_B2B-PH-K-S-LF-SN_B2B-PH-K-S-LF-SN_C131337.html"
+		(property "Datasheet" "https://lcsc.com/product-detail/C160352.html"
 			(at 171.45 99.06 0)
 			(hide yes)
@@
 			)
 		)
-		(property "Description" "Connector Header 2 position 2mm Pitch 2A Through Hole"
+		(property "Description" "Connector Header 2 position 2mm Pitch 2A SMD"
 			(at 171.45 86.36 0)
 			(hide yes)
@@
 			)
 		)
-		(property "MPN" "B2B-PH-K-S(LF)(SN)"
+		(property "MPN" "B2B-PH-SM4-TB(LF)(SN)"
 			(at 171.45 104.14 0)
 			(hide yes)
@@
 			)
 		)
-		(property "LCSC Part" "C131337"
+		(property "LCSC Part" "C160352"
 			(at 171.45 106.68 0)
 			(hide yes)
@@
 			)
 		)
-		(property "Value" "ZX-PZ1.27-2-5PZZ"
+		(property "Value" "HX PZ1.27-2x5P TP"
 			(at 215.9 74.93 0)
 			(show_name no)
@@
 			)
 		)
-		(property "Footprint" "easyeda2kicad:HDR-TH_10P-P1.27-V-M-R2-C5-S1.27"
+		(property "Footprint" "easyeda2kicad:HDR-SMD_10P-P1.27-V-M-R2-C5-LS5.5_1"
 			(at 215.9 97.79 0)
 			(hide yes)
@@
 			)
 		)
-		(property "Datasheet" "https://www.lcsc.com/datasheet/C7501289.pdf"
+		(property "Datasheet" "https://www.lcsc.com/datasheet/C41376037.pdf"
 			(at 215.9 100.33 0)
 			(hide yes)
@@
 			)
 		)
-		(property "Manufacturer" "Megastar(兆星)"
+		(property "Manufacturer" "hanxia"
 			(at 215.9 102.87 0)
 			(hide yes)
@@
 			)
 		)
-		(property "MPN" "ZX-PZ1.27-2-5PZZ"
+		(property "MPN" "HX PZ1.27-2x5P TP"
 			(at 215.9 105.41 0)
 			(hide yes)
@@
 			)
 		)
-		(property "LCSC Part" "C7501289"
+		(property "LCSC Part" "C41376037"
 			(at 215.9 107.95 0)
 			(hide yes)
@@
 			)
 		)
-		(property "Value" "R_Potentiometer_Trim"
+		(property "Value" "10k"
 			(at 394.97 76.1999 0)
 			(show_name no)
@@
 			)
 		)
-		(property "Footprint" "Potentiometer_THT:Potentiometer_Bourns_3296W_Vertical"
+		(property "Footprint" "easyeda2kicad:RES-ADJ-SMD_3P-L3.0-W3.8-P1.75-BR"
 			(at 397.51 74.93 0)
 			(hide yes)
@@
 			)
 		)
-		(property "Value" "0.8uF"
+		(property "Value" "0.8pF"
 			(at 234.95 187.96 90)
 			(show_name no)
@@
 			)
 		)
-		(property "Footprint" ""
+		(property "Footprint" "Resistor_SMD:R_0402_1005Metric"
 			(at 342.9 236.728 90)
 			(hide yes)
@@
 			)
 		)
-		(property "Footprint" "easyeda2kicad:IND-SMD_L4.0-W4.0_LQH44PN2R2MP0L"
+		(property "Footprint" "easyeda2kicad:IND-SMD_L4.0-W4.0"
 			(at 52.07 31.75 0)
 			(hide yes)
@@
 			)
 		)
-		(property "Value" "Conn_01x03_Pin"
+		(property "Value" "2.54-3P-LT"
 			(at 395.732 49.022 0)
 			(show_name no)
@@
 			)
 		)
-		(property "Footprint" "Connector_PinHeader_2.54mm:PinHeader_1x03_P2.54mm_Vertical"
+		(property "Footprint" "easyeda2kicad:CONN-SMD_2.54-3P-LT"
 			(at 392.43 54.61 0)
 			(hide yes)
@@
 			)
 		)
-		(property "Footprint" "easyeda2kicad:IND-SMD_L4.0-W4.0_LQH44PN2R2MP0L"
+		(property "Footprint" "easyeda2kicad:IND-SMD_L4.0-W4.0_NRS4018T"
 			(at 534.67 193.04 0)
 			(hide yes)
@@
 			)
 		)
-		(property "Footprint" ""
+		(property "Footprint" "Resistor_SMD:R_0402_1005Metric"
 			(at 342.9 241.808 90)
 			(hide yes)
@@
 			)
 		)
-		(property "Value" "0.5uF"
+		(property "Value" "0.6pF"
 			(at 254 187.96 90)
 			(show_name no)
@@
 			)
 		)
-		(property "Footprint" ""
+		(property "Footprint" "Resistor_SMD:R_0402_1005Metric"
 			(at 342.9 239.268 90)
 			(hide yes)
@@
 			)
 		)
-		(property "Footprint" "easyeda2kicad:IND-SMD_L4.0-W4.0_LQH44PN2R2MP0L"
+		(property "Footprint" "easyeda2kicad:IND-SMD_L4.0-W4.0_NRS4018T"
 			(at 426.72 198.12 0)
 			(hide yes)
@@
 			)
 		)
-		(property "Footprint" "easyeda2kicad:IND-SMD_L4.0-W4.0_LQH44PN2R2MP0L"
+		(property "Footprint" "easyeda2kicad:IND-SMD_L4.0-W4.0"
 			(at 52.07 80.01 0)
 			(hide yes)
@@
 			)
 		)
-		(property "Footprint" "easyeda2kicad:IND-SMD_L4.0-W4.0_LQH44PN2R2MP0L"
+		(property "Footprint" "easyeda2kicad:L0402-R-RD"
 			(at 247.65 184.15 0)
 			(hide yes)
@@
 			)
 		)
-		(property "Value" "ZX-PZ1.27-2-5PZZ"
+		(property "Value" "HX PZ1.27-2x5P TP"
 			(at 215.9 50.8 0)
 			(show_name no)
@@
 			)
 		)
-		(property "Footprint" "easyeda2kicad:HDR-TH_10P-P1.27-V-M-R2-C5-S1.27"
+		(property "Footprint" "easyeda2kicad:HDR-SMD_10P-P1.27-V-M-R2-C5-LS5.5_1"
 			(at 215.9 73.66 0)
 			(hide yes)
@@
 			)
 		)
-		(property "Datasheet" "https://www.lcsc.com/datasheet/C7501289.pdf"
+		(property "Datasheet" "https://www.lcsc.com/datasheet/C41376037.pdf"
 			(at 215.9 76.2 0)
 			(hide yes)
@@
 			)
 		)
-		(property "Manufacturer" "Megastar(兆星)"
+		(property "Manufacturer" "hanxia"
 			(at 215.9 78.74 0)
 			(hide yes)
@@
 			)
 		)
-		(property "MPN" "ZX-PZ1.27-2-5PZZ"
+		(property "MPN" "HX PZ1.27-2x5P TP"
 			(at 215.9 81.28 0)
 			(hide yes)
@@
 			)
 		)
-		(property "LCSC Part" "C7501289"
+		(property "LCSC Part" "C41376037"
 			(at 215.9 83.82 0)
 			(hide yes)
@@
 			)
 		)
-		(property "Value" "B4B-XH-A"
+		(property "Value" "SM04B-SRSS-TB"
 			(at 223.52 35.5599 0)
 			(show_name no)
@@
 			)
 		)
-		(property "Footprint" "easyeda2kicad:CONN-TH_B4B-XH-A-LF-SN"
+		(property "Footprint" "easyeda2kicad:CONN-SMD_4P-P1.00_SM04B-SRSS-TB-LF-SN"
 			(at 215.9 45.72 0)
 			(hide yes)
@@
 			)
 		)
-		(property "Datasheet" "https://lcsc.com/product-detail/_JST-Sales-America_B4B-XH-A-LF-SN_JST-Sales-America-B4B-XH-A-LF-SN_C144395.html"
+		(property "Datasheet" "https://lcsc.com/product-detail/C160404.html"
 			(at 215.9 48.26 0)
 			(hide yes)
@@
 			)
 		)
-		(property "MPN" "B4B-XH-A(LF)(SN)"
+		(property "MPN" "SM04B-SRSS-TB(LF)(SN)"
 			(at 215.9 53.34 0)
 			(hide yes)
@@
 			)
 		)
-		(property "LCSC Part" "C144395"
+		(property "LCSC Part" "C160404"
 			(at 215.9 55.88 0)
 			(hide yes)

Commit message: cleanup
Parts:
- C16, C18: value 10u -> 10uF
Changed lines of the file:
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@@
 			)
 		)
-		(property "Value" "10u"
+		(property "Value" "10uF"
 			(at 31.75 56.134 0)
 			(show_name no)
@@
 			)
 		)
-		(property "Value" "10u"
+		(property "Value" "10uF"
 			(at 31.75 104.394 0)
 			(show_name no)

Commit message: design support software
Parts:
- C1, C12, C13, C14, C15, C29, C30, C31, C32, C33, C4, C6, C8: LCSC Part (none) -> C307331
- C11, C2, C24, C3, C5: LCSC Part (none) -> C52923
- C16, C18, C20, C21, C22, C23, C7: LCSC Part (none) -> C15850
- C17, C19: LCSC Part (none) -> C52306
- C25: LCSC Part (none) -> C778333
- C26: LCSC Part (none) -> C3875120
- C27, C35: LCSC Part (none) -> C1547
- D1, D10, D11, D12, D6, D7, D8, D9: LCSC Part (none) -> C2843891
- D5: LCSC Part (none) -> C2827688
- J1: LCSC Part (none) -> C146125
- J2: LCSC Part (none) -> C2681544
- J3: LCSC Part (none) -> C266888
- L2, L3: LCSC Part (none) -> C2849472
- L4, L5: LCSC Part (none) -> C92959
- L6: LCSC Part (none) -> C86065
- P1: LCSC Part (none) -> C456012
- Q1, Q2, Q4: LCSC Part (none) -> C3018484
- Q3, Q5, Q6: LCSC Part (none) -> C8545
- R1: LCSC Part (none) -> C25792
- R10, R11, R12, R13, R14, R7, R8, R9: LCSC Part (none) -> C25169
- R15: LCSC Part (none) -> C25905
- R16, R17: LCSC Part (none) -> C100318
- R18, R23, R24: LCSC Part (none) -> C25076
- R19: LCSC Part (none) -> C159084
- R2: LCSC Part (none) -> C22369540
- R20, R22, R3, R4: LCSC Part (none) -> C49330233
- R21: LCSC Part (none) -> C64043
- R25: LCSC Part (none) -> C144809
- R26, R27: LCSC Part (none) -> C25900
- R28, R5, R6: LCSC Part (none) -> C25104
- RV1: LCSC Part (none) -> C719176
- SW1: LCSC Part (none) -> C139797
- TH1: LCSC Part (none) -> C77131
- U1: LCSC Part (none) -> C190794
- Y1: LCSC Part (none) -> C187794

Commit message: NPM revisions
Parts:
- removed C3: 1uF, Capacitor_SMD:C_0402_1005Metric, symbol Device:C
- removed C4: 100nF, Capacitor_SMD:C_0402_1005Metric, symbol Device:C
- removed CN1: B2B-PH-SM4-TB, easyeda2kicad:CONN-SMD_B2B-PH-SM4-TB-LF-SN, symbol easyeda2kicad:B2B-PH-K-S
- removed P1: USB_C_Plug_USB2.0, easyeda2kicad:TYPE-C-SMD_TYPE-C-6P_1, symbol Connector:USB_C_Plug_USB2.0
- removed TH1: Thermistor, Resistor_SMD:R_0402_1005Metric, symbol Device:Thermistor
- added C10: 2.2uF, Capacitor_SMD:C_0402_1005Metric, symbol Device:C
- added C9: 1uF, Capacitor_SMD:C_0805_2012Metric, symbol Device:C
- added CN1: B3B-PH-K-S, easyeda2kicad:CONN-TH_B3B-PH-K-S, symbol easyeda2kicad:B3B-PH-K-S
- added USB1: TYPE-C 16PIN 2MD, easyeda2kicad:USB-C-SMD_TYPE-C-16PIN-2MD-073, symbol easyeda2kicad:TYPE-C16PIN2MD
- R15: value 5.1k -> 10k; footprint Resistor_SMD:R_0402_1005Metric -> (none); LCSC Part C25905 -> (none)
- R16, R17: value 22R -> 10k; footprint Resistor_SMD:R_0402_1005Metric -> (none); LCSC Part C100318 -> (none)
- R2: value 150k -> 330k
Connections:
- net +1V8: now also R16.2, R17.2
- net +5V: no longer C5.1, D5.4 (VCC), U3.B1 (VBUS), U3.B2 (VBUS)
- net BIO_LS: now also C9.1
- net GND: now also C10.2, C9.2, CN1.3, USB1.13 (EH), USB1.14 (EH), USB1.A1B12 (GND), USB1.B1A12 (GND); no longer C23.1
- net NPM_SCL: now also R16.1
- net NPM_SDA: now also R17.1
- net USB_D+: now also USB1.A6 (Dp1), USB1.B6 (Dp2); no longer R16.2
- net USB_D-: now also USB1.A7 (Dn1), USB1.B7 (Dn2); no longer R17.2
- net NTC: now reaches U3.D3 (NTC)
- net NTC: now also CN1.2
- net CC2: now reaches U3.B3 (CC2)
- net CC2: now also USB1.B5 (CC2)
- net at U3.D1 (VBAT): now also U3.D2 (VBAT), C10.1
- net USB_CC: no longer names the net of R15.1
- net USB_CC: no longer U3.D5 (CC1)
- new net: C5.1, D5.4 (VCC), U3.B1 (VBUS), U3.B2 (VBUS), USB1.A4B9 (VBUS), USB1.B4A9 (VBUS)
- new net CC1: U3.D5 (CC1), USB1.A5 (CC1)
- no-connect marks 110 -> 108
Other:
- note added: "BUCK1 SUPPLY"
- note added: "BUCK2 SUPPLY"
- note added: "Battery JST 2.54mm 1x3P"
- note removed: "Battery JST 2.54mm 1x2P"
- moved on the sheet: C6, LED1

Commit message: nrf52840 changes, h-bridge update
Parts:
- removed Q2, Q4: BSS84, Package_TO_SOT_SMD:SOT-23, symbol Transistor_FET:BSS84
- removed Q5, Q6: 2N7002, Package_TO_SOT_SMD:SOT-23, symbol Transistor_FET:2N7002
- removed RV1: 10k, easyeda2kicad:RES-ADJ-SMD_3P-L3.0-W3.8-P1.75-BR, symbol Device:R_Potentiometer_Trim
- added C28: 1uF, Capacitor_SMD:C_0805_2012Metric, symbol Device:C
- added C3: 1nF, symbol Device:C
- added D2: BAV199DW, Package_TO_SOT_SMD:SOT-363_SC-70-6, symbol Diode:BAV199DW
- added R29: 100k, symbol Device:R
- added U5: DRV8871DDA, Package_SO:Texas_HTSOP-8-1EP_3.9x4.9mm_P1.27mm_EP2.95x4.9mm_Mask2.4x3.1mm_ThermalVias, symbol Driver_Motor:DRV8871DDA
- R15: value 10k -> 100k
- R23: value 100R -> 18k; footprint Resistor_SMD:R_0402_1005Metric -> (none); LCSC Part C25076 -> (none)
- R24: value 100R -> 1M; footprint Resistor_SMD:R_0402_1005Metric -> (none); LCSC Part C25076 -> (none)
Connections:
- net SIREN_FB is gone; now on net Strobe_In: U1.AC19 (P0.23)
- net +15V: now also U5.5 (VM)
- net +1V8: now also LED2.4 (+); no longer U11.1
- net +3.3V: no longer U14.1
- net ACC_INT1: now also U1.AC17 (P0.21); no longer U1.AD16 (P0.20)
- net ACC_INT2: now also U1.AD18 (P0.22); no longer U1.AC17 (P0.21)
- net ACC_SCL: now also U1.AD16 (P0.20); no longer U1.AC15 (P0.19)
- net ACC_SDA: now also U1.AC15 (P0.19); no longer U1.AD12 (P0.17)
- net GND: now also C24.2, R15.1, R23.2, C28.2, C3.2, D2.1 (A1), R29.1, U5.1 (GND), U5.7 (GND), U5.9 (GND); no longer C24.1, R15.2
- net NPM_INT: now also U1.AD12 (P0.17); no longer U1.AC11 (P0.16)
- net NPM_SCL: now also U1.AC11 (P0.16); no longer U1.AD10 (P0.15)
- net NPM_SDA: now also U1.AD10 (P0.15); no longer U1.AC9 (P0.14)
- net SIREN_PWM: now also U5.3 (IN1); no longer R23.1
- net SIREN_PWM_INVERTED: now also U5.2 (IN2); no longer R24.2
- net Strobe_In: no longer U1.AD18 (P0.22)
- net UART_RX: now also U1.AC9 (P0.14); no longer U1.AD8 (P0.13)
- net UART_TX: now also U1.AD8 (P0.13); no longer U1.U1 (TRACEDATA1/P0.12)
- net VSYS: no longer LED2.4 (+)
- net at J2.1 (Pin_1): now also U5.6 (OUT1)
- net VBUS: now reaches C5.1, D5.4 (VCC), U3.B1 (VBUS), U3.B2 (VBUS), USB1.A4B9 (VBUS), USB1.B4A9 (VBUS)
- net at R24.1: now also J2.2 (Pin_2)
- net at J2.3 (Pin_3): now also U5.8 (OUT2)
- net at C16.1, L2.1, U12.5 (IN): no longer U12.4 (EN)
- net at LED2.1 (R-): now also R5.2; no longer R28.2
- net at LED2.3 (B-): now also R28.2; no longer R5.2
- net at C18.1, L3.1, U13.5 (IN): no longer U13.4 (EN)
- net at R5.1: now also U1.A20 (P1.10); no longer U1.B11 (AIN4/P0.28)
- net ALARM_LS: now reaches U3.A5 (LSOUT2/VOUTLDO2)
- net ALARM_LS: now also R15.2, U12.4 (EN), U13.4 (EN), C28.1, R29.2
- net VBOUSOUT: now reaches U3.C3 (VBUSOUT)
- net VBOUSOUT: now also C24.1, U1.AD2 (VBUS)
- net at R28.1: now also U1.B17 (P1.12); no longer U1.B9 (AIN6/P0.30)
- net at R6.1: now also U1.B19 (P1.11); no longer U1.A10 (AIN5/P0.29)
- net PIEZO_FB: now reaches U1.A12 (AIN0/P0.02)
- net PIEZO_FB: now also R24.2, C3.1, D2.6 (K3A4)
- net VTref_52840: now reaches U1.U24 (P1.04)
- net VTref_52840: now also U14.1
- removed net +5V: C24.2, U1.AD2 (VBUS)
- new net: R23.1, U5.4 (ILIM)
- new net +3V3: D2.2 (K2)
- new net VTref_9151: U11.1
- no-connect marks 108 -> 104
Other:
- moved on the sheet: J2, LED2, R5

Commit message: RF
Parts:
- added C_ANT1, C_ANT2: DNP, Capacitor_SMD:C_01005_0402Metric, symbol Device:C
- added R30: 0R, Resistor_SMD:R_01005_0402Metric, symbol Device:R
- added U15: BWU.FL-IPEX1, easyeda2kicad:IPEX-SMD_BWIPX-1-001E, symbol easyeda2kicad:BWU.FL-IPEX1
- C12: value 100nF -> 1uF
- C25: value 0.6pF -> 0.5pF
Connections:
- net GND: now also C12.2, U1.B5 (DEC4), C_ANT1.2, C_ANT2.2, U15.2, U15.3
- net at L6.2, U1.H23 (ANT): now also C26.2; no longer C25.2
- new net: C_ANT2.1, R30.2, U15.1, U7.1
- new net RF: C25.2, C_ANT1.1, L6.1, R30.1
Other:
- note added: "RF SECTION"
- moved on the sheet: C12
