File: smart_pouch.kicad_sch (KiCad schematic)
At the start: 110 parts, among them CN1 B3B-PH-K-S, J1 XH-2P-SMD, J2 2.54-3P-LT, J3 SIM_Card, Q1 BSS84, Q3 2N7002, SW1 SW_Push, U1 nRF52840, U10 BWU.FL-IPEX1, U11 HX PZ1.27-2x5P TP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

Commit message: 52840 final + rf final
Parts:
- removed C14: 100nF, Capacitor_SMD:C_0402_1005Metric, symbol Device:C
- removed U15: BWU.FL-IPEX1, easyeda2kicad:IPEX-SMD_BWIPX-1-001E, symbol easyeda2kicad:BWU.FL-IPEX1
- added C34, C4: 12pF, symbol Device:C
- added TP1, TP2, TP3: TestPoint, symbol Connector:TestPoint
- added Y2: 32.768kHz, symbol Device:Crystal
- C11: value 1uF -> 100pF
- C13, C33: now not fitted; now left out of the parts list
- C15: value 100nF -> 4.7uF
Connections:
- net GND: now also U1.B3 (DCC), C34.2, C4.2, TP2.1, TP3.1
- net at C_ANT2.1, R30.2, U7.1: now also TP1.1
- net at U1.E24 (DEC6): now also C33.2, U1.A18 (DEC2)
- net at U1.D2 (XL1/P0.00): now also C4.1, Y2.2
- net at U1.F2 (XL2/P0.01): now also C34.1, Y2.1
- no-connect marks 104 -> 101

Commit message: LEDs
Parts:
- removed D12: LED, easyeda2kicad:LED-SMD_L3.0-W3.0_XL-3030UWC-1W-3V, symbol Device:LED
- removed Q1: BSS84, Package_TO_SOT_SMD:SOT-23, symbol Transistor_FET:BSS84
- removed R13, R14: 4.7, Resistor_SMD:R_0402_1005Metric, symbol Device:R
- added C14: 100nF, symbol Device:C
- added D4: LED, easyeda2kicad:LED-SMD_L3.0-W3.0_XL-3030UWC-1W-3V, symbol Device:LED
- added Q1: AO3400A, Package_TO_SOT_SMD:SOT-23, symbol Transistor_FET:AO3400A
- R10, R7, R8, R9: value 4.7 -> 39R; footprint Resistor_SMD:R_0402_1005Metric -> (none); LCSC Part C25169 -> (none)
- R11: value 4.7 -> 150R; footprint Resistor_SMD:R_0402_1005Metric -> (none); LCSC Part C25169 -> (none)
- R12: value 4.7 -> 10k; footprint Resistor_SMD:R_0402_1005Metric -> (none); LCSC Part C25169 -> (none)
Connections:
- net +12V: now also R10.1, R7.1, R8.1, R9.1
- net +15V: now also C14.1
- net +3.3V: no longer D1.2 (A), D10.2 (A), D11.2 (A), D6.2 (A), D7.2 (A), D8.2 (A), D9.2 (A)
- net GND: now also C14.2; no longer R10.2, R11.2, R7.2, R8.2, R9.2
- net Strobe_In: now also R11.1
- net at D9.1 (K): now also D8.2 (A); no longer R11.1
- net at D8.1 (K): now also R9.2; no longer R10.1
- net at R12.1: now also R11.2, Q1.1 (G); no longer D10.1 (K)
- net at D1.1 (K): now also D4.2 (A); no longer R7.1
- net at D7.1 (K): now also D6.2 (A); no longer R9.1
- net at D6.1 (K): now also R8.2; no longer R8.1
- net at D11.1 (K): now also D10.2 (A)
- new net: D1.2 (A), D11.2 (A), D7.2 (A), D9.2 (A), Q1.3 (D)
- new net: D4.1 (K), R7.2
- new net: D10.1 (K), R10.2
Other:
- note added: "drain"
- note added: "gate"
- note added: "source"
- moved on the sheet: D1, R26, R27, U4

Commit message: Piezo and strobe update
Parts:
- removed C3: 1nF, symbol Device:C
- removed D2: BAV199DW, Package_TO_SOT_SMD:SOT-363_SC-70-6, symbol Diode:BAV199DW
- removed Q1: AO3400A, Package_TO_SOT_SMD:SOT-23, symbol Transistor_FET:AO3400A
- removed R24: 1M, symbol Device:R
- added Q2: PMV20XNER, easyeda2kicad:SOT-23-3_L2.9-W1.3-P1.90-LS2.4-BR, symbol easyeda2kicad:PMV20XNER
- added R13: 560k, symbol Device:R
- added R14: 2.2M, symbol Device:R
Connections:
- net GND: now also Q2.2 (S), R13.2
- net PIEZO_FB: now also R13.1, R14.2
- net at J2.2 (Pin_2): now also R14.1
- net at R11.2, R12.1: now also Q2.1 (G)
- net at D1.2 (A), D11.2 (A), D7.2 (A)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: now also Q2.3 (D)
Other:
- note removed: "drain"
- note removed: "gate"
- note removed: "source"
- moved on the sheet: D1, D10, D11, D4, D6, D7, D8, D9, R10, R11, R12, R26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

Commit message: final revision
Parts:
- removed C1, C30: 100nF, Capacitor_SMD:C_0402_1005Metric, symbol Device:C
- removed D3: SP3012-04UTG, easyeda2kicad:UDFN-10_L2.5-W1.0-P0.50-BL, symbol easyeda2kicad:SP3012-04UTG
- added C3, C36: 100nF, symbol Device:C
- U9: footprint easyeda2kicad:CONN-SMD_4P-P1.00_SM04B-SRSS-TB-LF-SN -> easyeda2kicad:CONN-TH_B4B-XH-A-LF-SN; LCSC Part C160404 -> C144395; MPN SM04B-SRSS-TB(LF)(SN) -> B4B-XH-A(LF)(SN)
Connections:
- net +1V8: now also C3.1, C36.1; no longer C29.2, U2.65 (VDD_GPIO), U9.2
- net GND: now also C23.1, C3.2, C36.2
- net VTref_9151: now also C29.2, U2.65 (VDD_GPIO), U9.2
Other:
- note added: "Andrew Suggs"
- note added: "Final"
- note added: "June 18th, 2026"
- note added: "Travel Vault"
- note added: "nRF52840 AQFN"
- note removed: "nRF52840 BLE"
- moved on the sheet: C14, C28, CN1, D1, D10, D11, D13, D4, D6, D7, D8, D9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

Commit message: gpt-footprint-bom-run
Parts:
- C13, C_ANT1: now in the parts list
- C14, C3, C34, C36, C4: footprint (none) -> Capacitor_SMD:C_0402_1005Metric
- J1: LCSC Part C146125 -> C722696
- J2: LCSC Part C2681544 -> C722698
- R10, R7, R8, R9: footprint (none) -> Resistor_SMD:R_2512_6332Metric
- R11, R12, R13, R14, R15, R16, R17, R23, R29: footprint (none) -> Resistor_SMD:R_0402_1005Metric
- R30: LCSC Part (none) -> C364372; MPN (none) -> RC0100JR-070RL; Manufacturer (none) -> YAGEO
- TP1, TP2, TP3: footprint (none) -> TestPoint:TestPoint_Pad_D1.0mm; now left out of the parts list
- U2: symbol easyeda2kicad:NRF9151-SICA -> easyeda2kicad:NRF9151-LACA-R7; MPN nRF9151-SICA -> nRF9151-LACA-R7
- U5: LCSC Part (none) -> C75864; MPN (none) -> DRV8871DDAR; Manufacturer (none) -> Texas Instruments
- U9: value SM04B-SRSS-TB -> XH-4A; LCSC Part C144395 -> C2908602; MPN B4B-XH-A(LF)(SN) -> XH-4A; Manufacturer JST -> HCTL
- Y2: footprint (none) -> Crystal:Crystal_SMD_3215-2Pin_3.2x1.5mm
Changed lines of the file:
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@@
 			)
 		)
-		(property "Footprint" ""
+		(property "Footprint" "Capacitor_SMD:C_0402_1005Metric"
 			(at 436.5752 107.95 0)
 			(hide yes)
@@
 			)
 		)
+		(property "Manufacturer" "YAGEO"
+			(at 0 0 0)
+			(hide yes)
+			(show_name no)
+			(do_not_autoplace no)
+			(effects
+				(font
+					(size 1.27 1.27)
+				)
+			)
+		)
+		(property "MPN" "RC0100JR-070RL"
+			(at 0 0 0)
+			(hide yes)
+			(show_name no)
+			(do_not_autoplace no)
+			(effects
+				(font
+					(size 1.27 1.27)
+				)
+			)
+		)
+		(property "LCSC Part" "C364372"
+			(at 0 0 0)
+			(hide yes)
+			(show_name no)
+			(do_not_autoplace no)
+			(effects
+				(font
+					(size 1.27 1.27)
+				)
+			)
+		)
 		(pin "2"
 		)
@@
 			)
 		)
-		(property "LCSC Part" "C146125"
+		(property "LCSC Part" "C722696"
 			(at 16.51 -1.27 0)
 			(hide yes)
@@
 	)
 	(symbol
-		(lib_id "easyeda2kicad:NRF9151-SICA")
+		(lib_id "easyeda2kicad:NRF9151-LACA-R7")
 		(at 96.52 232.41 0)
 		(unit 1)
@@
 			)
 		)
-		(property "MPN" "nRF9151-SICA"
+		(property "MPN" "nRF9151-LACA-R7"
 			(at 96.52 318.77 0)
 			(hide yes)
@@
 			)
 		)
-		(property "Footprint" ""
+		(property "Footprint" "Resistor_SMD:R_0402_1005Metric"
 			(at 438.912 60.96 90)
 			(hide yes)
@@
 			)
 		)
-		(property "Footprint" ""
+		(property "Footprint" "Resistor_SMD:R_0402_1005Metric"
 			(at 512.572 156.21 90)
 			(hide yes)
@@
 		(body_style 1)
 		(exclude_from_sim no)
-		(in_bom yes)
+		(in_bom no)
 		(on_board yes)
 		(in_pos_files yes)
@@
 			)
 		)
-		(property "Footprint" ""
+		(property "Footprint" "TestPoint:TestPoint_Pad_D1.0mm"
 			(at 528.32 35.56 0)
 			(hide yes)
@@
 			)
 		)
-		(property "Footprint" ""
+		(property "Footprint" "Resistor_SMD:R_0402_1005Metric"
 			(at 438.912 50.8 90)
 			(hide yes)
@@
 		(body_style 1)
 		(exclude_from_sim yes)
-		(in_bom no)
+		(in_bom yes)
 		(on_board yes)
 		(in_pos_files yes)
@@
 		(body_style 1)
 		(exclude_from_sim no)
-		(in_bom yes)
+		(in_bom no)
 		(on_board yes)
 		(in_pos_files yes)
@@
 			)
 		)
-		(property "Footprint" ""
+		(property "Footprint" "TestPoint:TestPoint_Pad_D1.0mm"
 			(at 532.13 35.56 0)
 			(hide yes)
@@
 			)
 		)
-		(property "Footprint" ""
+		(property "Footprint" "Capacitor_SMD:C_0402_1005Metric"
 			(at 374.65 170.4848 0)
 			(hide yes)
@@
 			)
 		)
-		(property "Footprint" ""
+		(property "Footprint" "Capacitor_SMD:C_0402_1005Metric"
 			(at 393.3952 100.33 0)
 			(hide yes)
@@
 			)
 		)
-		(property "Footprint" ""
+		(property "Footprint" "Resistor_SMD:R_0402_1005Metric"
 			(at 499.872 156.21 90)
 			(hide yes)
@@
 			)
 		)
-		(property "LCSC Part" "C2681544"
+		(property "LCSC Part" "C722698"
 			(at 821.69 -12.7 0)
 			(hide yes)
@@
 			)
 		)
-		(property "Footprint" ""
+		(property "Footprint" "Resistor_SMD:R_0402_1005Metric"
 			(at 323.342 71.12 90)
 			(hide yes)
@@
 		(body_style 1)
 		(exclude_from_sim yes)
-		(in_bom no)
+		(in_bom yes)
 		(on_board yes)
 		(in_pos_files yes)
@@
 			)
 		)
-		(property "Footprint" ""
+		(property "Footprint" "Crystal:Crystal_SMD_3215-2Pin_3.2x1.5mm"
 			(at 359.41 166.37 0)
 			(hide yes)
@@
 			)
 		)
-		(property "Footprint" ""
+		(property "Footprint" "Resistor_SMD:R_2512_6332Metric"
 			(at 353.822 36.83 90)
 			(hide yes)
@@
 			)
 		)
-		(property "Footprint" ""
+		(property "Footprint" "Capacitor_SMD:C_0402_1005Metric"
 			(at 389.89 30.1752 0)
 			(hide yes)
@@
 			)
 		)
+		(property "Manufacturer" "Texas Instruments"
+			(at 0 0 0)
+			(hide yes)
+			(show_name no)
+			(do_not_autoplace no)
+			(effects
+				(font
+					(size 1.27 1.27)
+				)
+			)
+		)
+		(property "MPN" "DRV8871DDAR"
+			(at 0 0 0)
+			(hide yes)
+			(show_name no)
+			(do_not_autoplace no)
+			(effects
+				(font
+					(size 1.27 1.27)
+				)
+			)
+		)
+		(property "LCSC Part" "C75864"
+			(at 0 0 0)
+			(hide yes)
+			(show_name no)
+			(do_not_autoplace no)
+			(effects
+				(font
+					(size 1.27 1.27)
+				)
+			)
+		)
 		(pin "4"
 		)
@@
 			)
 		)
-		(property "Footprint" ""
+		(property "Footprint" "Resistor_SMD:R_0402_1005Metric"
 			(at 317.5 62.738 90)
 			(hide yes)
@@
 			)
 		)
-		(property "Footprint" ""
+		(property "Footprint" "Resistor_SMD:R_0402_1005Metric"
 			(at 38.862 41.91 90)
 			(hide yes)
@@
 			)
 		)
-		(property "Footprint" ""
+		(property "Footprint" "Resistor_SMD:R_2512_6332Metric"
 			(at 336.042 36.83 90)
 			(hide yes)
@@
 			)
 		)
-		(property "Footprint" ""
+		(property "Footprint" "Resistor_SMD:R_0402_1005Metric"
 			(at 38.862 90.17 90)
 			(hide yes)
@@
 			)
 		)
-		(property "Footprint" ""
+		(property "Footprint" "Resistor_SMD:R_2512_6332Metric"
 			(at 348.742 36.83 90)
 			(hide yes)
@@
 			)
 		)
-		(property "Footprint" ""
+		(property "Footprint" "Resistor_SMD:R_0402_1005Metric"
 			(at 405.892 53.34 90)
 			(hide yes)
@@
 		(body_style 1)
 		(exclude_from_sim no)
-		(in_bom yes)
+		(in_bom no)
 		(on_board yes)
 		(in_pos_files yes)
@@
 			)
 		)
-		(property "Footprint" ""
+		(property "Footprint" "TestPoint:TestPoint_Pad_D1.0mm"
 			(at 529.59 36.83 0)
 			(hide yes)
@@
 			)
 		)
-		(property "Footprint" ""
+		(property "Footprint" "Resistor_SMD:R_2512_6332Metric"
 			(at 342.392 36.83 90)
 			(hide yes)
@@
 			)
 		)
-		(property "Footprint" ""
+		(property "Footprint" "Capacitor_SMD:C_0402_1005Metric"
 			(at 374.65 161.5948 0)
 			(hide yes)
@@
 			)
 		)
-		(property "Value" "SM04B-SRSS-TB"
+		(property "Value" "XH-4A"
 			(at 242.57 34.2899 0)
 			(show_name no)
@@
 			)
 		)
-		(property "Datasheet" "https://lcsc.com/product-detail/_JST-Sales-America_B4B-XH-A-LF-SN_JST-Sales-America-B4B-XH-A-LF-SN_C144395.html"
+		(property "Datasheet" ""
 			(at 234.95 46.99 0)
 			(hide yes)
@@
 			)
 		)
-		(property "Manufacturer" "JST"
+		(property "Manufacturer" "HCTL"
 			(at 234.95 49.53 0)
 			(hide yes)
@@
 			)
 		)
-		(property "MPN" "B4B-XH-A(LF)(SN)"
+		(property "MPN" "XH-4A"
 			(at 234.95 52.07 0)
 			(hide yes)
@@
 			)
 		)
-		(property "LCSC Part" "C144395"
+		(property "LCSC Part" "C2908602"
 			(at 234.95 54.61 0)
 			(hide yes)

Commit message: Initial PCB commit
Parts:
- removed J3: SIM_Card, easyeda2kicad:SIM-SMD_SMN-303, symbol Connector:SIM_Card
- removed R3, R4: 10k, Resistor_SMD:R_0402_1005Metric, symbol Device:R
- added C37: 100nF, Capacitor_SMD:C_0402_1005Metric, symbol Device:C
- added Card1: SMN-303, easyeda2kicad:SIM-SMD_SMN-303, symbol easyeda2kicad:SMN-303
- added R31: 10k, Resistor_SMD:R_0402_1005Metric, symbol Device:R
- TP1, TP2, TP3: footprint TestPoint:TestPoint_Pad_D1.0mm -> TestPoint:TestPoint_Pad_1.0x1.0mm
Connections:
- net +1V8: now also R31.2
- net GND: now also C37.2, Card1.10 (EP), Card1.11 (EP), Card1.8 (EP), Card1.9 (EP), Card1.C5 (GND)
- net SIM_1V8: now also C37.1, Card1.C1 (VCC)
- net SIM_CLK: now also Card1.C3 (CLK)
- net SIM_IO: now also Card1.C7 (I/O), R31.1
- net SIM_RST: now also Card1.C2 (RST)
- net SIM_CD: now reaches U2.26 (SIM_DET)
- net SIM_CD: now also Card1.CD
- no-connect marks 101 -> 100

Commit message: pcb basic layout
Parts:
- CN1: value B3B-PH-K-S -> JST 1x3 Battery P=1.27mm; Manufacturer JST -> JST 1x3 Battery P=1.27mm
- D5: value PRTR5V0U2X -> PRTR5V0U2X ESD
- J1: value XH-2P-SMD -> Solenoid XH-2P-SMD
- J2: value 2.54-3P-LT -> 2.54-3P-LT Piezo
- LED1: value 19-237/R6GHBHC-A01/2T -> Power RGB
- LED2: value 19-237/R6GHBHC-A01/2T -> USER LED
- U11: value HX PZ1.27-2x5P TP -> 9151 SWD P=1.27mm 2x5P
- U14: value HX PZ1.27-2x5P TP -> 52840 SWD P=1.27mm 2x5P
- U8: value SEN0348_CONN -> JST P=1mm 01x06
- U9: value XH-4A -> XH-4A UART 9151
- USB1: value TYPE-C 16PIN 2MD -> TYPE-C 16P
Changed lines of the file:
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@@
 			)
 		)
-		(property "Value" "XH-2P-SMD"
+		(property "Value" "Solenoid XH-2P-SMD"
 			(at 288.29 64.77 0)
 			(show_name no)
@@
 			)
 		)
-		(property "Value" "PRTR5V0U2X"
+		(property "Value" "PRTR5V0U2X ESD"
 			(at 480.06 275.5198 0)
 			(show_name no)
@@
 			)
 		)
-		(property "Value" "19-237/R6GHBHC-A01/2T"
+		(property "Value" "Power RGB"
 			(at 405.765 143.51 0)
 			(show_name no)
@@
 			)
 		)
-		(property "Value" "HX PZ1.27-2x5P TP"
+		(property "Value" "52840 SWD P=1.27mm 2x5P"
 			(at 234.95 73.66 0)
 			(show_name no)
@@
 			)
 		)
-		(property "Description" ""
+		(property "Description" "52840 SWD P=1.27mm 2x5P"
 			(at 234.95 83.82 0)
 			(hide yes)
@@
 			)
 		)
-		(property "Value" "19-237/R6GHBHC-A01/2T"
+		(property "Value" "USER LED"
 			(at 360.045 261.62 0)
 			(show_name no)
@@
 			)
 		)
-		(property "Value" "2.54-3P-LT"
+		(property "Value" "2.54-3P-LT Piezo"
 			(at 425.958 36.322 0)
 			(show_name no)
@@
 			)
 		)
-		(property "Description" "Generic connector, single row, 01x03, script generated"
+		(property "Description" "Piezo"
 			(at 429.26 41.91 0)
 			(hide yes)
@@
 			)
 		)
-		(property "Value" "TYPE-C 16PIN 2MD"
+		(property "Value" "TYPE-C  16P"
 			(at 532.13 269.24 0)
 			(show_name no)
@@
 			)
 		)
-		(property "Value" "SEN0348_CONN"
+		(property "Value" "JST P=1mm 01x06"
 			(at 324.358 49.276 0)
 			(hide yes)
@@
 			)
 		)
-		(property "Value" "B3B-PH-K-S"
+		(property "Value" "JST 1x3 Battery P=1.27mm"
 			(at 191.77 82.5499 0)
 			(hide yes)
@@
 			)
 		)
-		(property "Description" ""
+		(property "Description" "JST 1x3 Battery P=1.27mm"
 			(at 186.69 81.28 0)
 			(hide yes)
@@
 			)
 		)
-		(property "Manufacturer" "JST"
+		(property "Manufacturer" "JST 1x3 Battery P=1.27mm"
 			(at 186.69 96.52 0)
 			(hide yes)
@@
 			)
 		)
-		(property "Value" "HX PZ1.27-2x5P TP"
+		(property "Value" "9151 SWD P=1.27mm 2x5P"
 			(at 234.95 49.53 0)
 			(show_name no)
@@
 			)
 		)
-		(property "Description" ""
+		(property "Description" "9151 SWD P=1.27mm 2x5P"
 			(at 234.95 59.69 0)
 			(hide yes)
@@
 			)
 		)
-		(property "Value" "XH-4A"
+		(property "Value" "XH-4A UART 9151"
 			(at 242.57 34.2899 0)
 			(show_name no)
@@
 			)
 		)
-		(property "Description" ""
+		(property "Description" "XH-4A UART 9151"
 			(at 234.95 33.02 0)
 			(hide yes)

Commit message: replace npm13100 package
Parts:
- removed C23: 10uF, Capacitor_SMD:C_0805_2012Metric, symbol Device:C
- removed CN1: JST 1x3 Battery P=1.27mm, easyeda2kicad:CONN-TH_B3B-PH-K-S, symbol easyeda2kicad:B3B-PH-K-S
- removed U3: NPM1300, easyeda2kicad:BGA-35_L3.1-W2.4-R5-C7-P0.42_NPM1300-CAAA-R, symbol easyeda2kicad:NPM1300-CAAA-R7
- added C30: 10uF, Capacitor_SMD:C_0805_2012Metric, symbol Device:C
- added CN2: B2B-PH-K-S, easyeda2kicad:CONN-TH_B2B-PH-K-S, symbol easyeda2kicad:B2B-PH-K-S
- added U15: NPM1300-QEAA-R7, footprints2:QFN32_5X5_NOR, symbol 2026-06-18_20-37-18:NPM1300-QEAA-R7
Connections:
- net +1V8: now also C7.1, R16.1, U15.1 (VOUT1), U15.12 (VDDIO); no longer C7.2, R16.2
- net +3.3V: now also C30.1, U15.28 (LSIN1/VINLDO1), U15.32 (VOUT2)
- net ALARM_LS: now also U15.31 (LSOUT2/VOUTLDO2)
- net BIO_LS: now also U15.29 (LSOUT1/VOUTLDO1)
- net CC1: now also U15.23 (CC1)
- net CC2: now also U15.24 (CC2)
- net GND: now also C7.2, C30.2, CN2.2, U15.2 (PVSS1), U15.33 (AVSS), U15.6 (PVSS2); no longer C7.1
- net NPM_INT: now also U15.8 (GPIO1)
- net NPM_RESET: now also U15.7 (GPIO0)
- net NPM_SCL: now also R16.2, U15.14 (SCL); no longer R16.1
- net NPM_SDA: now also U15.13 (SDA)
- net VBOUSOUT: now also U15.22 (VBUSOUT)
- net VBUS: now also U15.21 (VBUS)
- net VSYS: now also U15.20 (VSYS), U15.4 (PVDD)
- net at SW1.1: now also U15.15 (SHPHLD)
- net at LED1.1 (R-): now also U15.25 (LED0)
- net at LED1.2 (G-): now also LED1.3 (B-), U15.26 (LED1), U15.27 (LED2)
- net FB: now reaches J2.2 (Pin_2), R14.1
- net at R2.1: now also U15.16 (VSET2)
- net +: now reaches J2.1 (Pin_1), U5.6 (OUT1)
- net -: now reaches J2.3 (Pin_3), U5.8 (OUT2)
- net at L4.2: now also U15.3 (SW1)
- net at L5.2: now also U15.5 (SW2)
- net at C10.1: now also U15.19 (VBAT)
- net at R1.1: now also U15.17 (VSET1)
- no-connect marks 100 -> 102
Other:
- note removed: "+"
- note removed: "-"
- note removed: "FB"
- note removed: "Status LED"
